Commit message: add fusion policy

File: resources/tita/urdf/tita_description.urdf (robot description, URDF)
Before this commit: robot tita_ros2_control, 14 links, 13 joints
Links:
- link left_leg_2: geometry collision box size=0.2 0.09 0.05; visual mesh filename=../meshes/left_leg_2.STL
- link right_leg_2: geometry collision box size=0.2 0.09 0.05; visual mesh filename=../meshes/right_leg_2.STL
Joints:
- joint joint_left_leg_1: limit lower=-0.785398 upper=0.785398 effort=45 velocity=25 -> lower=-0.785398 upper=0.785398 effort=60 velocity=25
- joint joint_left_leg_2: limit lower=-1.919862 upper=3.490659 effort=45 velocity=25 -> lower=-1.919862 upper=3.490659 effort=60 velocity=25
- joint joint_left_leg_3: limit lower=-2.670354 upper=-0.698132 effort=45 velocity=25 -> lower=-2.670354 upper=-0.698132 effort=60 velocity=25
- joint joint_right_leg_1: limit lower=-0.785398 upper=0.785398 effort=45 velocity=25 -> lower=-0.785398 upper=0.785398 effort=60 velocity=25
- joint joint_right_leg_2: limit lower=-1.919862 upper=3.490659 effort=45 velocity=25 -> lower=-1.919862 upper=3.490659 effort=60 velocity=25
- joint joint_right_leg_3: limit lower=-2.670354 upper=-0.698132 effort=45 velocity=25 -> lower=-2.670354 upper=-0.698132 effort=60 velocity=25

Commit message: 新增逐际动力轮腿模型

File: resources/tita/urdf/tita_description.urdf (robot description, URDF)
Before this commit: robot tita_ros2_control, 14 links, 13 joints
Links:
- added link imu_link, mass 0.001; collision box size=.001 .001 .001; visual box size=0.001 0.001 0.001
- link base_link: mass 13.2 -> 11.36226789
- link left_leg_2: mass 3.0984 -> 3.018005; geometry visual mesh filename=../meshes/left_leg_2.STL
- link right_leg_2: mass 3.0987 -> 3.018005; geometry visual mesh filename=../meshes/right_leg_2.STL
Joints:
- added joint imu_joint: type fixed, parent base_link, child imu_link, origin xyz=0 0 0 rpy=0 0 0
- joint joint_left_leg_1: limit lower=-0.785398 upper=0.785398 effort=60 velocity=25 -> lower=-0.785398 upper=0.785398 effort=80 velocity=15
- joint joint_left_leg_2: limit lower=-1.919862 upper=3.490659 effort=60 velocity=25 -> lower=-1.919862 upper=3.490659 effort=60 velocity=15
- joint joint_left_leg_3: limit lower=-2.670354 upper=-0.698132 effort=60 velocity=25 -> lower=-2.670354 upper=-0.698132 effort=60 velocity=15
- joint joint_left_leg_4: limit lower=-999999 upper=999999 effort=15 velocity=20 -> lower=-6.283185e4 upper=6.283185e4 effort=10 velocity=50
- joint joint_right_leg_1: limit lower=-0.785398 upper=0.785398 effort=60 velocity=25 -> lower=-0.785398 upper=0.785398 effort=80 velocity=15
- joint joint_right_leg_2: limit lower=-1.919862 upper=3.490659 effort=60 velocity=25 -> lower=-1.919862 upper=3.490659 effort=60 velocity=15
- joint joint_right_leg_3: limit lower=-2.670354 upper=-0.698132 effort=60 velocity=25 -> lower=-2.670354 upper=-0.698132 effort=60 velocity=15
- joint joint_right_leg_4: limit lower=-999999 upper=999999 effort=15 velocity=20 -> lower=-6.283185e4 upper=6.283185e4 effort=10 velocity=50
